File: hardware/magicmouth-v0.1-ds.sch (EAGLE design)
At the start: 38 parts, among them IC1 LM386N, IC2 ATMEGA328P_PDIP, Q1 16Mhz, U1 ARDUINOR3-NOIOREF-NOTEXT

Commit message: trace corrections
Connections:
- net N$24 renamed D8
Changed lines of the file:
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@@
 <instance part="JP8" gate="A" x="276.86" y="38.1"/>
 <instance part="U$2" gate="G$1" x="111.76" y="40.64" rot="R180"/>
-<instance part="JP9" gate="G$1" x="254" y="58.42" rot="R90"/>
+<instance part="JP9" gate="G$1" x="254" y="58.42" smashed="yes" rot="R90">
+<attribute name="NAME" x="250.698" y="55.88" size="1.778" layer="95" rot="R90"/>
+</instance>
 <instance part="R7" gate="G$1" x="40.64" y="83.82" rot="R270"/>
 <instance part="PAD1" gate="P" x="60.96" y="71.12"/>
@@
 </segment>
 </net>
-<net name="N$24" class="0">
-<segment>
-<wire x1="228.6" y1="83.82" x2="302.26" y2="83.82" width="0.1524" layer="91"/>
-<pinref part="JP3" gate="G$1" pin="1"/>
-<pinref part="IC2" gate="G$1" pin="PB0(ICP)"/>
-</segment>
-</net>
 <net name="SIGNAL" class="0">
-<segment>
-<label x="274.32" y="81.28" size="1.778" layer="95"/>
-<wire x1="228.6" y1="81.28" x2="302.26" y2="81.28" width="0.1524" layer="91"/>
-<pinref part="JP3" gate="G$1" pin="2"/>
-<pinref part="IC2" gate="G$1" pin="PB1(OC1A)"/>
-</segment>
 <segment>
 <pinref part="R2" gate="G$1" pin="1"/>
@@
 <label x="38.1" y="124.46" size="1.778" layer="95" rot="R90"/>
 </segment>
+<segment>
+<pinref part="JP3" gate="G$1" pin="2"/>
+<pinref part="IC2" gate="G$1" pin="PB1(OC1A)"/>
+<wire x1="228.6" y1="81.28" x2="302.26" y2="81.28" width="0.1524" layer="91"/>
+<label x="274.32" y="81.28" size="1.778" layer="95"/>
+</segment>
 </net>
 <net name="MISO" class="0">
 <segment>
-<wire x1="228.6" y1="73.66" x2="289.56" y2="73.66" width="0.1524" layer="91"/>
 <label x="274.32" y="73.66" size="1.778" layer="95"/>
 <pinref part="JP6" gate="A" pin="2"/>
@@
 <wire x1="289.56" y1="40.64" x2="289.56" y2="73.66" width="0.1524" layer="91"/>
 <pinref part="IC2" gate="G$1" pin="PB4(MISO)"/>
+<wire x1="289.56" y1="73.66" x2="228.6" y2="73.66" width="0.1524" layer="91"/>
 </segment>
 </net>
 <net name="SCK" class="0">
 <segment>
-<wire x1="228.6" y1="71.12" x2="287.02" y2="71.12" width="0.1524" layer="91"/>
 <label x="274.32" y="71.12" size="1.778" layer="95"/>
 <pinref part="JP5" gate="A" pin="2"/>
@@
 <wire x1="287.02" y1="43.18" x2="287.02" y2="71.12" width="0.1524" layer="91"/>
 <pinref part="IC2" gate="G$1" pin="PB5(SCK)"/>
+<wire x1="287.02" y1="71.12" x2="228.6" y2="71.12" width="0.1524" layer="91"/>
 </segment>
 </net>
@@
 <net name="MOSI" class="0">
 <segment>
-<wire x1="228.6" y1="76.2" x2="292.1" y2="76.2" width="0.1524" layer="91"/>
 <label x="274.32" y="76.2" size="1.778" layer="95"/>
 <pinref part="JP7" gate="A" pin="2"/>
@@
 <wire x1="292.1" y1="38.1" x2="292.1" y2="76.2" width="0.1524" layer="91"/>
 <pinref part="IC2" gate="G$1" pin="PB3(MOSI/OC2)"/>
+<wire x1="292.1" y1="76.2" x2="228.6" y2="76.2" width="0.1524" layer="91"/>
 </segment>
 </net>
@@
 <segment>
 <pinref part="JP9" gate="G$1" pin="1"/>
-<wire x1="228.6" y1="78.74" x2="254" y2="78.74" width="0.1524" layer="91"/>
 <wire x1="254" y1="78.74" x2="254" y2="66.04" width="0.1524" layer="91"/>
 <pinref part="IC2" gate="G$1" pin="PB2(SS/OC1B)"/>
+<wire x1="254" y1="78.74" x2="228.6" y2="78.74" width="0.1524" layer="91"/>
 </segment>
 </net>
@@
 </segment>
 </net>
+<net name="D8" class="0">
+<segment>
+<pinref part="IC2" gate="G$1" pin="PB0(ICP)"/>
+<pinref part="JP3" gate="G$1" pin="1"/>
+<wire x1="302.26" y1="83.82" x2="228.6" y2="83.82" width="0.1524" layer="91"/>
+</segment>
+</net>
