File: hardware/magicmouth-v1.0.brd (EAGLE design)
At the start: 100 x 80 mm, 110 parts, among them IC1 LM386N, IC2 ATMEGA328P_PDIP, Q1 16Mhz, U1 ARDUINOR3-NOIOREF-NOTEXT

Commit message: 10uf bypass cap for LM386
Parts:
- removed PAD5, PAD6: (no value), wirepad:1,6/0,8
- added C11: 22pF, rcl:C025-025X050
- C4: value 47nF -> 10uF; device rcl:C050-025X075 -> rcl:E2,5-7
- C5: value 220uF -> 47nF; device rcl:TT2D7 -> rcl:C050-025X075
- C7: value 100nF -> 220uF; device rcl:C025-025X050 -> rcl:TT2D7
- C9: value 22pF -> 100nF
- moved C7 49.4 mm to (18.5, 24.1), turned to 180 degrees
- moved C6 23.8 mm to (22.2, 47.6), turned to 180 degrees
- moved C9 20.3 mm to (55.1, 29.7), turned to 315 degrees
- moved C4 19.1 mm to (43.2, 39.4), turned to 180 degrees
- moved C8 15.2 mm to (64.8, 41.3), turned to 135 degrees
- moved C5 8.47 mm to (24.1, 39.4), turned to 270 degrees
- moved C10 5.33 mm to (64.8, 47.5)
- moved IC1 1.27 mm to (31.8, 43.2)
- moved PAD1 1.27 mm to (38.1, 47.0)
- moved PAD2 1.27 mm to (38.1, 44.5)
- moved PAD3 1.27 mm to (38.1, 39.4)
- moved PAD4 1.27 mm to (38.1, 41.9)
- moved C3 0.64 mm to (27.7, 55.2), turned to 180 degrees
Connections:
- removed net N$94: IC1.7, PAD5.1
- new net N$24: C4.+, IC1.7
- net +5V: now also C8.1; no longer C7.1
- net GND: now also C10.1, C11.2, C4.-, C7.-, C9.2; no longer C10.2, C6.-, C7.2, C9.1
- net N$1: now also C5.1, C6.+; no longer C4.1, C5.+, PAD6.1
- net N$11: now also C11.1; no longer C10.1
- net N$3: now also C9.1; no longer C8.1
- net N$4: now also C5.2; no longer C4.2
- net N$6: now also C10.2; no longer C9.2
- net N$8: now also C6.-; no longer C5.-
- net VCC: now also C7.+; no longer C6.+
Routing:
- net GND: track 201.7 -> 217.0 mm, vias 4 -> 2
- net N$24: track 0.00 -> 14.3 mm
- net N$9: track 30.3 -> 26.4 mm, vias 2 -> 1
- net N$1: track 14.1 -> 10.8 mm
- net N$8: track 22.8 -> 20.2 mm
- net N$94: track 2.54 -> 0.00 mm
- net N$87: track 7.04 -> 4.98 mm
- net VCC: track 59.9 -> 58.2 mm, vias 2 -> 0
- net SCK: track 28.2 -> 29.3 mm
- net MISO: track 23.3 -> 22.8 mm
